Commit message: turned off infra1 and infra2

File: urdf/_d405.gazebo.xacro (robot description, xacro)
@@ -6,5 +6,5 @@
 -->
 <robot xmlns:xacro="http://ros.org/wiki/xacro">
-  <xacro:macro name="gazebo_d405" params="camera_name reference_link topics_ns depth_optical_frame color_optical_frame infrared1_optical_frame infrared2_optical_frame publish_pointcloud:=true" >
+  <xacro:macro name="gazebo_d405" params="camera_name reference_link topics_ns depth_optical_frame color_optical_frame publish_pointcloud:=true" >
     <!-- Load parameters to model's main link-->
     <xacro:property name="deg_to_rad" value="0.01745329251994329577" />
@@ -63,5 +63,5 @@
           </noise>
         </camera>
-        <always_on>1</always_on>
+        <always_on>0</always_on>
         <update_rate>30</update_rate>
         <visualize>0</visualize>
@@ -85,5 +85,5 @@
           </noise>
         </camera>
-        <always_on>1</always_on>
+        <always_on>0</always_on>
         <update_rate>30</update_rate>
         <visualize>0</visualize>
@@ -116,13 +116,11 @@
         <depthUpdateRate>30.0</depthUpdateRate>
         <colorUpdateRate>30.0</colorUpdateRate>
-        <infraredUpdateRate>30.0</infraredUpdateRate>
+        <infraredUpdateRate>0.0</infraredUpdateRate>
         <depthTopicName>depth/image_raw</depthTopicName>
         <colorTopicName>color/image_raw</colorTopicName>
-        <infrared1TopicName>infra1/image_raw</infrared1TopicName>
-        <infrared2TopicName>infra2/image_raw</infrared2TopicName>
+        <!-- <infrared1TopicName>infra1/'image_raw'</infrared1TopicName> -->
+        <!-- <infrared2TopicName>infra2/image_raw</infrared2TopicName> -->
         <colorOpticalframeName>${color_optical_frame}</colorOpticalframeName>
         <depthOpticalframeName>${depth_optical_frame}</depthOpticalframeName>
-        <infrared1OpticalframeName>${infrared1_optical_frame}</infrared1OpticalframeName>
-        <infrared2OpticalframeName>${infrared2_optical_frame}</infrared2OpticalframeName>
         <rangeMinDepth>0.07</rangeMinDepth>
         <rangeMaxDepth>1.0</rangeMaxDepth>
